File: DMH_Mixer_PCB/DMH_Mixer_PCB.kicad_pcb (KiCad board)
At the start: 2 copper layers, 48 x 175 mm, 0 parts

Commit message: PCB work in progress
Parts:
- added C1: 47uF, Capacitor_THT:CP_Radial_D5.0mm_P2.00mm, F.Cu at (166.5, 100.2)
- added C2: 47uF, Capacitor_THT:CP_Radial_D5.0mm_P2.00mm, F.Cu at (166.5, 106.8)
- added C3: 100nF, Capacitor_THT:C_Disc_D4.3mm_W1.9mm_P5.00mm, F.Cu at (157.6, 98.7)
- added C4: 100nF, Capacitor_THT:C_Disc_D4.3mm_W1.9mm_P5.00mm, F.Cu at (157.6, 102.1)
- added C5: 100nF, Capacitor_THT:C_Disc_D4.3mm_W1.9mm_P5.00mm, F.Cu at (157.6, 105.6)
- added C6: 100nF, Capacitor_THT:C_Disc_D4.3mm_W1.9mm_P5.00mm, F.Cu at (157.6, 109.0)
- added D1: 1N4148, Diode_THT:D_DO-35_SOD27_P7.62mm_Horizontal, F.Cu at (171.2, 44.6)
- added D2: 1N4148, Diode_THT:D_DO-35_SOD27_P7.62mm_Horizontal, F.Cu at (171.2, 48.2)
- added D4: SB140-, Diode_THT:D_DO-41_SOD81_P10.16mm_Horizontal, F.Cu at (157.9, 90.6)
- added D5: SB140+, Diode_THT:D_DO-41_SOD81_P10.16mm_Horizontal, F.Cu at (157.9, 94.8)
- added J0: Conn_01x01, Connector_PinHeader_2.54mm:PinHeader_1x01_P2.54mm_Vertical, F.Cu at (166.5, 112.4)
- added J1: TS_Jack_6.35mm_Sw, SynthStuff:CUI_MJ-63052A, F.Cu at (58.5, 190.2)
- added J100: IDC_02x05, SynthStuff:IDC-Header_2x05_P2.54mm_Vertical_Eurorack, B.Cu at (92.0, 49.1)
- added J2: TS_Jack_6.35mm_Sw, SynthStuff:CUI_MJ-63052A, F.Cu at (75.0, 190.2)
- added J3: TS_Jack_6.35mm_Sw, SynthStuff:CUI_MJ-63052A, F.Cu at (91.5, 190.2)
- added J4: TS_Jack_6.35mm_Sw, SynthStuff:CUI_MJ-63052A, F.Cu at (58.5, 208.8)
- added J5: TS_Jack_6.35mm_Sw, SynthStuff:CUI_MJ-63052A, F.Cu at (75.0, 208.8)
- added J50: Conn_01x06, Connector_PinHeader_2.54mm:PinHeader_1x06_P2.54mm_Vertical, B.Cu at (57.0, 162.8)
- added J51: Conn_01x06, Connector_PinHeader_2.54mm:PinHeader_1x06_P2.54mm_Vertical, B.Cu at (39.0, 159.6)
- added J6: TS_Jack_6.35mm_Sw, SynthStuff:CUI_MJ-63052A, F.Cu at (91.5, 208.8)
- added J7: IDC_02x05, SynthStuff:IDC-Header_2x05_P2.54mm_Vertical_BackBone, B.Cu at (57.0, 175.5)
- added R1: 100k, Resistor_THT:R_Axial_DIN0207_L6.3mm_D2.5mm_P7.62mm_Horizontal, F.Cu at (160.4, 33.0)
- added R10: 100k, Resistor_THT:R_Axial_DIN0207_L6.3mm_D2.5mm_P7.62mm_Horizontal, F.Cu at (160.4, 69.5)
- added R11: 27k, Resistor_THT:R_Axial_DIN0207_L6.3mm_D2.5mm_P7.62mm_Horizontal, F.Cu at (160.4, 73.5)
- added R12: 1k, Resistor_THT:R_Axial_DIN0207_L6.3mm_D2.5mm_P7.62mm_Horizontal, F.Cu at (160.4, 77.6)
- added R2: 100k, Resistor_THT:R_Axial_DIN0207_L6.3mm_D2.5mm_P7.62mm_Horizontal, F.Cu at (160.4, 37.1)
- added R3: 100k, Resistor_THT:R_Axial_DIN0207_L6.3mm_D2.5mm_P7.62mm_Horizontal, F.Cu at (160.4, 41.1)
- added R4: 100k, Resistor_THT:R_Axial_DIN0207_L6.3mm_D2.5mm_P7.62mm_Horizontal, F.Cu at (160.4, 45.2)
- added R5: 100k, Resistor_THT:R_Axial_DIN0207_L6.3mm_D2.5mm_P7.62mm_Horizontal, F.Cu at (160.4, 49.2)
- added R6: 100k, Resistor_THT:R_Axial_DIN0207_L6.3mm_D2.5mm_P7.62mm_Horizontal, F.Cu at (160.4, 53.3)
- added R7: 1k, Resistor_THT:R_Axial_DIN0207_L6.3mm_D2.5mm_P7.62mm_Horizontal, F.Cu at (160.4, 57.3)
- added R8: 1k, Resistor_THT:R_Axial_DIN0207_L6.3mm_D2.5mm_P7.62mm_Horizontal, F.Cu at (160.4, 61.4)
- added R9: 100k, Resistor_THT:R_Axial_DIN0207_L6.3mm_D2.5mm_P7.62mm_Horizontal, F.Cu at (160.4, 65.4)
- added RV1: 100k, Potentiometer_THT:Potentiometer_Alpha_RD901F-40-00D_Single_Vertical, F.Cu at (72.5, 66.0)
- added RV2: 100k, Potentiometer_THT:Potentiometer_Alpha_RD901F-40-00D_Single_Vertical, F.Cu at (72.5, 101.7)
- added RV3: 100k, Potentiometer_THT:Potentiometer_Alpha_RD901F-40-00D_Single_Vertical, F.Cu at (72.5, 137.5)
- added RV4: 20k, Potentiometer_THT:Potentiometer_Alpha_RD901F-40-00D_Single_Vertical, F.Cu at (80.5, 171.7)
- added U1: TL074, Package_DIP:DIP-14_W7.62mm_Socket, B.Cu at (63.8, 80.0)

Commit message: Component placing in progress
Parts:
- removed J7: IDC_02x05, SynthStuff:IDC-Header_2x05_P2.54mm_Vertical_BackBone
- added J200: IDC_02x05, SynthStuff:IDC-Header_2x05_P2.54mm_Vertical_BackBone, B.Cu at (58.1, 166.8)
- added J60: Conn_01x06, Connector_PinHeader_2.54mm:PinHeader_1x06_P2.54mm_Vertical, B.Cu at (54.4, 179.5)
- added J61: Conn_01x06, Connector_PinSocket_2.54mm:PinSocket_1x06_P2.54mm_Vertical, F.Cu at (29.1, 184.8)
- C1, C2, C3, C4, C5, C6, D1, D2, D4, D5, R1, R10, R11, R12, R2, R3, R4, R5, R6, R7, R8, R9: moved to B.Cu
- J51: footprint Connector_PinHeader_2.54mm:PinHeader_1x06_P2.54mm_Vertical -> Connector_PinSocket_2.54mm:PinSocket_1x06_P2.54mm_Vertical; moved to F.Cu
- moved C1 122.8 mm to (55.5, 47.8), turned to 90 degrees
- moved J0 111.3 mm to (57.2, 91.0)
- moved D5 104.9 mm to (61.2, 54.1), turned to 90 degrees
- moved C6 95.3 mm to (63.5, 124.5), turned to 180 degrees
- moved C2 94.4 mm to (94.5, 45.8), turned to -90 degrees
- moved C3 94.2 mm to (63.5, 103.5), turned to 180 degrees
- moved D4 83.6 mm to (88.5, 43.9), turned to -90 degrees
- moved D1 68.2 mm to (103.6, 35.3), turned to 180 degrees
- moved D2 68.2 mm to (103.6, 38.9), turned to 180 degrees
- moved C4 67.9 mm to (94.9, 75.9), turned to 180 degrees
- moved C5 67.9 mm to (94.9, 79.3), turned to 180 degrees
- moved R1 46.9 mm to (114.4, 23.7), turned to 180 degrees
- moved R10 46.9 mm to (114.4, 60.1), turned to 180 degrees
- moved R11 46.9 mm to (114.4, 64.2), turned to 180 degrees
- moved R12 46.9 mm to (114.4, 68.2), turned to 180 degrees
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Connections:
- J2 pad TN: Net-(J51-Pin_1) -> Net-(J61-Pin_2)
- J50 pad 1: /Inputs and Outputs/Input 1 Jack -> /Core Circuit/Input 1
- J50 pad 2: /Inputs and Outputs/Input 2 Jack -> /Core Circuit/Input 2
- J50 pad 3: /Inputs and Outputs/Input 3 Jack -> /Core Circuit/Input 3
- J50 pad 4: /Inputs and Outputs/Output - Jack -> /Core Circuit/Clipped Output
- J50 pad 5: /Inputs and Outputs/Output + Jack -> /Core Circuit/Output -
- J50 pad 6: /Inputs and Outputs/Output Clipped -> /Core Circuit/Output +

Commit message: Finished main PCB
Parts:
- removed J1, J2, J3, J4, J5, J6: TS_Jack_6.35mm_Sw, SynthStuff:CUI_MJ-63052A
- removed J51, J61: Conn_01x06, Connector_PinSocket_2.54mm:PinSocket_1x06_P2.54mm_Vertical
- J50, J60: value Conn_01x06 -> Conn_01x08; footprint Connector_PinHeader_2.54mm:PinHeader_1x06_P2.54mm_Vertical -> Connector_PinSocket_2.54mm:PinSocket_1x08_P2.54mm_Vertical
- moved D1 122.9 mm to (86.8, 157.0)
- moved R7 117.4 mm to (97.2, 164.2), turned to -90 degrees
- moved D2 115.3 mm to (79.2, 151.5), turned to 0 degrees
- moved R8 114.0 mm to (94.0, 164.2), turned to -90 degrees
- moved R12 98.8 mm to (90.8, 164.2), turned to -90 degrees
- moved R10 94.5 mm to (58.5, 136.3), turned to 90 degrees
- moved R11 82.1 mm to (63.5, 128.7), turned to -90 degrees
- moved R5 80.2 mm to (71.2, 107.5), turned to 0 degrees
- moved R6 78.6 mm to (78.8, 114.0)
- moved R9 73.6 mm to (78.8, 120.5)
- moved R4 65.8 mm to (71.2, 85.5), turned to 0 degrees
- moved R3 60.3 mm to (78.8, 80.5)
- moved R2 59.5 mm to (78.8, 75.5)
- moved R1 58.8 mm to (78.8, 70.5)
- moved J0 49.1 mm to (55.0, 140.0)
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Routing:
- net /Core Circuit/Input 1: track 0.00 -> 127.0 mm
- net -12V: track 0.00 -> 122.1 mm
- net Net-(R6-Pad2): track 0.00 -> 84.0 mm
- net /Core Circuit/Input 2: track 0.00 -> 80.9 mm
- net Net-(U1D--): track 0.00 -> 77.5 mm
- net +12V: track 0.00 -> 76.1 mm
- net Net-(R10-Pad2): track 0.00 -> 61.3 mm
- net Net-(R3-Pad1): track 0.00 -> 58.6 mm
- net Net-(D1-A): track 0.00 -> 55.5 mm
- net /Core Circuit/Input 3: track 0.00 -> 49.5 mm
- net Net-(U1D-+): track 0.00 -> 42.7 mm
- net Net-(U1A--): track 0.00 -> 41.1 mm
- net Net-(R2-Pad1): track 0.00 -> 27.8 mm
- net Net-(U1C--): track 0.00 -> 23.7 mm
- net Net-(U1B--): track 0.00 -> 22.6 mm
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- added copper zone on B.Cu, net GND
- added copper zone on F.Cu, net GND
Other:
- board size 48 x 175 mm -> 48 x 138 mm

Commit message: Finished connectors PCB
Routing:
- net -12V: track 122.1 -> 123.1 mm
- net Net-(R10-Pad2): track 61.3 -> 62.0 mm
Changed lines of the file:
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@@
 		(tags "Diode DO-35_SOD27 series Axial Horizontal pin pitch 7.62mm  length 4mm diameter 2mm")
 		(property "Reference" "D2"
-			(at 9.81 0 360)
+			(at 9.81 0 0)
 			(layer "B.SilkS")
 			(effects
@@
 		)
 		(property "Value" "1N4148"
-			(at 3.81 -2 360)
+			(at 3.81 -2 0)
 			(layer "B.SilkS")
 			(effects
@@
 		)
 		(fp_text user "K"
-			(at -1.69 0 360)
+			(at -1.69 0 0)
 			(layer "B.SilkS")
 			(effects
@@
 		)
 		(fp_text user "${REFERENCE}"
-			(at 4.11 0 360)
+			(at 4.11 0 0)
 			(layer "B.Fab")
 			(effects
@@
 		)
 		(fp_text user "K"
-			(at 0 1.8 360)
+			(at 0 1.8 0)
 			(layer "B.Fab")
 			(effects
@@
 		(tags "C Disc series Radial pin pitch 5.00mm  diameter 4.3mm width 1.9mm Capacitor")
 		(property "Reference" "C3"
-			(at 2.5 2 360)
+			(at 2.5 2 0)
 			(layer "B.SilkS")
 			(effects
@@
 		)
 		(property "Value" "100nF"
-			(at 3 0 360)
+			(at 3 0 0)
 			(layer "B.SilkS")
 			(effects
@@
 		)
 		(fp_text user "${REFERENCE}"
-			(at 2.5 0 360)
+			(at 2.5 0 0)
 			(layer "B.Fab")
 			(effects
@@
 		(tags "Resistor Axial_DIN0207 series Axial Horizontal pin pitch 7.62mm 0.25W = 1/4W length 6.3mm diameter 2.5mm")
 		(property "Reference" "R1"
-			(at 3.81 2.37 360)
+			(at 3.81 2.37 0)
 			(layer "B.SilkS")
 			(effects
@@
 		)
 		(property "Value" "100k"
-			(at 3.81 0 360)
+			(at 3.81 0 0)
 			(layer "B.SilkS")
 			(effects
@@
 		)
 		(fp_text user "${REFERENCE}"
-			(at 3.81 0 360)
+			(at 3.81 0 0)
 			(layer "B.Fab")
 			(effects
@@
 		(tags "THT DIP DIL PDIP 2.54mm 7.62mm 300mil Socket")
 		(property "Reference" "U1"
-			(at 8.3 2.33 360)
+			(at 8.3 2.33 0)
 			(layer "B.SilkS")
 			(effects
@@
 		)
 		(property "Value" "TL074"
-			(at 3.81 -17.57 360)
+			(at 3.81 -17.57 0)
 			(layer "B.Fab")
 			(effects
@@
 		)
 		(fp_text user "${REFERENCE}"
-			(at 3.81 -7.62 360)
+			(at 3.81 -7.62 0)
 			(layer "B.Fab")
 			(effects
@@
 		(tags "Resistor Axial_DIN0207 series Axial Horizontal pin pitch 7.62mm 0.25W = 1/4W length 6.3mm diameter 2.5mm")
 		(property "Reference" "R5"
-			(at 3.81 -2.25 360)
+			(at 3.81 -2.25 0)
 			(layer "B.SilkS")
 			(effects
@@
 		)
 		(property "Value" "100k"
-			(at 3.81 0 360)
+			(at 3.81 0 0)
 			(layer "B.SilkS")
 			(effects
@@
 		)
 		(fp_text user "${REFERENCE}"
-			(at 3.81 0 360)
+			(at 3.81 0 0)
 			(layer "B.Fab")
 			(effects
@@
 		(tags "Resistor Axial_DIN0207 series Axial Horizontal pin pitch 7.62mm 0.25W = 1/4W length 6.3mm diameter 2.5mm")
 		(property "Reference" "R9"
-			(at 3.81 2.37 360)
+			(at 3.81 2.37 0)
 			(layer "B.SilkS")
 			(effects
@@
 		)
 		(property "Value" "100k"
-			(at 3.81 0 360)
+			(at 3.81 0 0)
 			(layer "B.SilkS")
 			(effects
@@
 		)
 		(fp_text user "${REFERENCE}"
-			(at 3.81 0 360)
+			(at 3.81 0 0)
 			(layer "B.Fab")
 			(effects
@@
 		)
 		(fp_text user "${REFERENCE}"
-			(at 1.27 -5.08 360)
+			(at 1.27 -5.08 0)
 			(layer "B.Fab")
 			(effects
@@
 		(tags "Resistor Axial_DIN0207 series Axial Horizontal pin pitch 7.62mm 0.25W = 1/4W length 6.3mm diameter 2.5mm")
 		(property "Reference" "R4"
-			(at 3.81 -2.25 360)
+			(at 3.81 -2.25 0)
 			(layer "B.SilkS")
 			(effects
@@
 		)
 		(property "Value" "100k"
-			(at 3.81 0 360)
+			(at 3.81 0 0)
 			(layer "B.SilkS")
 			(effects
@@
 		)
 		(fp_text user "${REFERENCE}"
-			(at 3.81 0 360)
+			(at 3.81 0 0)
 			(layer "B.Fab")
 			(effects
@@
 	)
 	(gr_rect
-		(start 70 212.75)
-		(end 80 214.75)
+		(start 94 126.25)
+		(end 96 136.25)
 		(stroke
 			(width 0.1)
@@
 	)
 	(gr_text "Mk1.0 - Month Year"
-		(at 74.75 216.25 0)
+		(at 97.5 131.5 90)
 		(layer "B.SilkS")
 		(effects
@@
 	)
 	(segment
-		(start 61.25 101.25)
-		(end 63.5 103.5)
+		(start 55.5 47.75)
+		(end 55.5 52.5)
 		(width 1)
 		(layer "B.Cu")
@@
 	)
 	(segment
-		(start 57.92 54.58)
+		(start 55.5 52.5)
 		(end 57.75 54.75)
 		(width 1)
@@
 	)
 	(segment
-		(start 57.75 50)
-		(end 55.5 47.75)
+		(start 61.25 54.58)
+		(end 63.5 56.83)
 		(width 1)
 		(layer "B.Cu")
@@
 	)
 	(segment
-		(start 61.25 54.58)
-		(end 61.25 101.25)
+		(start 57.92 54.58)
+		(end 57.75 54.75)
 		(width 1)
 		(layer "B.Cu")
@@
 	)
 	(segment
-		(start 61.25 54.58)
-		(end 57.92 54.58)
+		(start 63.5 56.83)
+		(end 63.5 103.5)
 		(width 1)
 		(layer "B.Cu")
@@
 	)
 	(segment
-		(start 57.75 54.75)
-		(end 57.75 50)
+		(start 61.25 54.58)
+		(end 57.92 54.58)
 		(width 1)
 		(layer "B.Cu")
@@
 	)
 	(segment
-		(start 59.299999 123.700001)
-		(end 59.299999 116.114999)
+		(start 88.67 54.5)
+		(end 68.5 54.5)
 		(width 1)
 		(layer "F.Cu")
@@
 	)
 	(segment
-		(start 59.299999 116.114999)
-		(end 57.18 113.995)
+		(start 56.559315 124.5)
+		(end 58.5 124.5)
 		(width 1)
 		(layer "F.Cu")
@@
 	)
 	(segment
-		(start 88.67 54.5)
-		(end 68.5 54.5)
+		(start 88.75 54.58)
+		(end 88.67 54.5)
 		(width 1)
 		(layer "F.Cu")
@@
 	(segment
 		(start 58.5 124.5)
-		(end 59.299999 123.700001)
+		(end 60.5 122.5)
 		(width 1)
 		(layer "F.Cu")
@@
 	)
 	(segment
-		(start 56.559315 124.5)
-		(end 58.5 124.5)
-		(width 1)
-		(layer "F.Cu")
-		(net 3)
-	)
-	(segment
-		(start 88.75 54.58)
-		(end 88.67 54.5)
+		(start 54.5 102.5)
+		(end 54.5 122.440685)
 		(width 1)
 		(layer "F.Cu")
@@
 	)
 	(segment
-		(start 54.5 102.5)
-		(end 54.5 122.440685)
+		(start 60.5 122.5)
+		(end 60.5 117.315)
 		(width 1)
 		(layer "F.Cu")
@@
 	)
 	(segment
+		(start 60.5 117.315)
+		(end 57.18 113.995)
+		(width 1)
+		(layer "F.Cu")
+		(net 3)
+	)
+	(segment
 		(start 92.08 54.58)
 		(end 92.25 54.75)
@@
 	)
 	(segment
-		(start 92.25 54.75)
-		(end 92.25 50)
+		(start 88.75 54.58)
+		(end 92.08 54.58)
 		(width 1)
 		(layer "B.Cu")
@@
 	)
 	(segment
-		(start 92.25 50)
-		(end 94.5 47.75)
+		(start 94.5 52.5)
+		(end 92.25 54.75)
 		(width 1)
 		(layer "B.Cu")
@@
 	)
 	(segment
-		(start 88.75 54.58)
-		(end 92.08 54.58)
+		(start 94.5 47.75)
+		(end 94.5 52.5)
 		(width 1)
 		(layer "B.Cu")
@@
 	)
 	(segment
-		(start 79.75 141.75)
-		(end 90.75 152.75)
+		(start 90.75 151.5)
+		(end 90.75 164.19)
 		(width 0.2)
 		(layer "B.Cu")
@@
 	)
 	(segment
-		(start 90.75 152.75)
-		(end 90.75 164.19)
+		(start 57.18 127.37)
+		(end 58.5 128.69)
 		(width 0.2)
 		(layer "B.Cu")
@@
 	)
 	(segment
-		(start 57.18 127.37)
-		(end 58.5 128.69)
+		(start 81 141.75)
+		(end 90.75 151.5)
 		(width 0.2)
 		(layer "B.Cu")
@@
 	)
 	(segment
-		(start 58.5 128.69)
-		(end 58.69 128.69)
+		(start 71.75 141.75)
+		(end 81 141.75)
 		(width 0.2)
 		(layer "B.Cu")
@@
 	)
 	(segment
-		(start 71.75 141.75)
-		(end 79.75 141.75)
+		(start 58.5 128.69)
+		(end 58.69 128.69)
 		(width 0.2)
 		(layer "B.Cu")

Commit message: Updated fps with their 3D models
Parts:
- RV1, RV2, RV3, RV4: footprint Potentiometer_THT:Potentiometer_Alpha_RD901F-40-00D_Single_Vertical -> SynthStuff:Potentiometer_Alpha_RD901F-40-00D_Single_Vertical
Changed lines of the file:
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@@
 	(net 28 "Net-(J200-Pin_1)")
 	(net 29 "Net-(J200-Pin_2)")
-	(footprint "Potentiometer_THT:Potentiometer_Alpha_RD901F-40-00D_Single_Vertical"
+	(footprint "SynthStuff:Potentiometer_Alpha_RD901F-40-00D_Single_Vertical"
 		(locked yes)
 		(layer "F.Cu")
@@
 		(tags "potentiometer vertical 9mm single")
 		(property "Reference" "RV1"
-			(at 6.71 -4.64 90)
+			(at 6.71 -4.64 -90)
 			(layer "F.SilkS")
 			(effects
@@
 		)
 		(property "Value" "100k"
-			(at 0 9.86 90)
-			(layer "F.Fab")
-			(effects
-				(font
-					(size 1 1)
-					(thickness 0.15)
-				)
-			)
-		)
-		(property "Footprint" "Potentiometer_THT:Potentiometer_Alpha_RD901F-40-00D_Single_Vertical"
+			(at 2.725 8.5 270)
+			(layer "F.SilkS")
+			(effects
+				(font
+					(size 1 1)
+					(thickness 0.15)
+				)
+			)
+		)
+		(property "Footprint" "SynthStuff:Potentiometer_Alpha_RD901F-40-00D_Single_Vertical"
 			(at 0 0 90)
 			(unlocked yes)
@@
 			)
 		)
-		(property "Function" ""
-			(at 0 0 90)
-			(unlocked yes)
-			(layer "F.Fab")
-			(hide yes)
-			(effects
-				(font
-					(size 1 1)
-					(thickness 0.15)
-				)
+		(property "Function" "Input 1 Gain"
+			(at 2.475 2.5 180)
+			(layer "B.SilkS")
+			(effects
+				(font
+					(size 1 1)
+					(thickness 0.15)
+					(italic yes)
+				)
+				(justify mirror)
 			)
 		)
@@
 		)
 		(model "${KICAD8_3DMODEL_DIR}/Potentiometer_THT.3dshapes/Potentiometer_Alpha_RD901F-40-00D_Single_Vertical.wrl"
+			(hide yes)
 			(offset
 				(xyz 0 0 0)
@@
 			)
 		)
+		(model "${KIPRJMOD}/Libraries/SynthStuff/3D_models/ALPHA-RD901F-40.step"
+			(offset
+				(xyz 7.35 -2.5 0)
+			)
+			(scale
+				(xyz 1 1 1)
+			)
+			(rotate
+				(xyz 0 0 90)
+			)
+		)
+		(model "${KIPRJMOD}/Libraries/SynthStuff/3D_models/rk09l12d0a1w.stp"
+			(hide yes)
+			(offset
+				(xyz 7.5 -2.5 6.7)
+			)
+			(scale
+				(xyz 1 1 1)
+			)
+			(rotate
+				(xyz 0 180 90)
+			)
+		)
 	)
-	(footprint "Potentiometer_THT:Potentiometer_Alpha_RD901F-40-00D_Single_Vertical"
+	(footprint "SynthStuff:Potentiometer_Alpha_RD901F-40-00D_Single_Vertical"
 		(locked yes)
 		(layer "F.Cu")
@@
 		(tags "potentiometer vertical 9mm single")
 		(property "Reference" "RV4"
-			(at 6.71 -4.64 90)
+			(at 6.71 -4.64 -90)
 			(layer "F.SilkS")
 			(effects
@@
 		)
 		(property "Value" "20k"
-			(at 0 9.86 90)
-			(layer "F.Fab")
-			(effects
-				(font
-					(size 1 1)
-					(thickness 0.15)
-				)
-			)
-		)
-		(property "Footprint" "Potentiometer_THT:Potentiometer_Alpha_RD901F-40-00D_Single_Vertical"
+			(at -0.525 7.75 0)
+			(layer "F.SilkS")
+			(effects
+				(font
+					(size 1 1)
+					(thickness 0.15)
+				)
+			)
+		)
+		(property "Footprint" "SynthStuff:Potentiometer_Alpha_RD901F-40-00D_Single_Vertical"
 			(at 0 0 90)
 			(unlocked yes)
@@
 					(thickness 0.15)
 				)
+			)
+		)
+		(property "Function" "Clipping Amount"
+			(at 2.725 2.5 180)
+			(layer "B.SilkS")
+			(effects
+				(font
+					(size 1 1)
+					(thickness 0.15)
+					(italic yes)
+				)
+				(justify mirror)
 			)
 		)
@@
 		)
 		(model "${KICAD8_3DMODEL_DIR}/Potentiometer_THT.3dshapes/Potentiometer_Alpha_RD901F-40-00D_Single_Vertical.wrl"
+			(hide yes)
 			(offset
 				(xyz 0 0 0)
@@
 			(rotate
 				(xyz 0 0 0)
+			)
+		)
+		(model "${KIPRJMOD}/Libraries/SynthStuff/3D_models/ALPHA-RD901F-40.step"
+			(offset
+				(xyz 7.35 -2.5 0)
+			)
+			(scale
+				(xyz 1 1 1)
+			)
+			(rotate
+				(xyz 0 0 90)
+			)
+		)
+		(model "${KIPRJMOD}/Libraries/SynthStuff/3D_models/rk09l12d0a1w.stp"
+			(hide yes)
+			(offset
+				(xyz 7.5 -2.5 6.7)
+			)
+			(scale
+				(xyz 1 1 1)
+			)
+			(rotate
+				(xyz 0 180 90)
 			)
 		)
@@
 		)
 	)
-	(footprint "Potentiometer_THT:Potentiometer_Alpha_RD901F-40-00D_Single_Vertical"
+	(footprint "SynthStuff:Potentiometer_Alpha_RD901F-40-00D_Single_Vertical"
 		(locked yes)
 		(layer "F.Cu")
@@
 		(tags "potentiometer vertical 9mm single")
 		(property "Reference" "RV2"
-			(at 6.71 -4.64 90)
+			(at 6.71 -4.64 -90)
 			(layer "F.SilkS")
 			(effects
@@
 		)
 		(property "Value" "100k"
-			(at 0 9.86 90)
-			(layer "F.Fab")
-			(effects
-				(font
-					(size 1 1)
-					(thickness 0.15)
-				)
-			)
-		)
-		(property "Footprint" "Potentiometer_THT:Potentiometer_Alpha_RD901F-40-00D_Single_Vertical"
+			(at 2.725 8.5 270)
+			(layer "F.SilkS")
+			(effects
+				(font
+					(size 1 1)
+					(thickness 0.15)
+				)
+			)
+		)
+		(property "Footprint" "SynthStuff:Potentiometer_Alpha_RD901F-40-00D_Single_Vertical"
 			(at 0 0 90)
 			(unlocked yes)
@@
 			)
 		)
-		(property "Function" ""
-			(at 0 0 90)
-			(unlocked yes)
-			(layer "F.Fab")
-			(hide yes)
-			(effects
-				(font
-					(size 1 1)
-					(thickness 0.15)
-				)
+		(property "Function" "Input 2 Gain"
+			(at 2.475 2.5 180)
+			(layer "B.SilkS")
+			(effects
+				(font
+					(size 1 1)
+					(thickness 0.15)
+					(italic yes)
+				)
+				(justify mirror)
 			)
 		)
@@
 		)
 		(model "${KICAD8_3DMODEL_DIR}/Potentiometer_THT.3dshapes/Potentiometer_Alpha_RD901F-40-00D_Single_Vertical.wrl"
+			(hide yes)
 			(offset
 				(xyz 0 0 0)
@@
 			)
 		)
+		(model "${KIPRJMOD}/Libraries/SynthStuff/3D_models/ALPHA-RD901F-40.step"
+			(offset
+				(xyz 7.35 -2.5 0)
+			)
+			(scale
+				(xyz 1 1 1)
+			)
+			(rotate
+				(xyz 0 0 90)
+			)
+		)
+		(model "${KIPRJMOD}/Libraries/SynthStuff/3D_models/rk09l12d0a1w.stp"
+			(hide yes)
+			(offset
+				(xyz 7.5 -2.5 6.7)
+			)
+			(scale
+				(xyz 1 1 1)
+			)
+			(rotate
+				(xyz 0 180 90)
+			)
+		)
 	)
-	(footprint "Potentiometer_THT:Potentiometer_Alpha_RD901F-40-00D_Single_Vertical"
+	(footprint "SynthStuff:Potentiometer_Alpha_RD901F-40-00D_Single_Vertical"
 		(locked yes)
 		(layer "F.Cu")
@@
 		(tags "potentiometer vertical 9mm single")
 		(property "Reference" "RV3"
-			(at 6.71 -4.64 90)
+			(at 6.71 -4.64 -90)
 			(layer "F.SilkS")
 			(effects
@@
 		)
 		(property "Value" "100k"
-			(at 0 9.86 90)
-			(layer "F.Fab")
-			(effects
-				(font
-					(size 1 1)
-					(thickness 0.15)
-				)
-			)
-		)
-		(property "Footprint" "Potentiometer_THT:Potentiometer_Alpha_RD901F-40-00D_Single_Vertical"
+			(at 2.475 8.5 270)
+			(layer "F.SilkS")
+			(effects
+				(font
+					(size 1 1)
+					(thickness 0.15)
+				)
+			)
+		)
+		(property "Footprint" "SynthStuff:Potentiometer_Alpha_RD901F-40-00D_Single_Vertical"
 			(at 0 0 90)
 			(unlocked yes)
@@
 					(thickness 0.15)
 				)
+			)
+		)
+		(property "Function" "Input 3 Gain"
+			(at 2.475 2.5 180)
+			(layer "B.SilkS")
+			(effects
+				(font
+					(size 1 1)
+					(thickness 0.15)
+					(italic yes)
+				)
+				(justify mirror)
 			)
 		)
@@
 		)
 		(model "${KICAD8_3DMODEL_DIR}/Potentiometer_THT.3dshapes/Potentiometer_Alpha_RD901F-40-00D_Single_Vertical.wrl"
+			(hide yes)
 			(offset
 				(xyz 0 0 0)
@@
 			)
 		)
+		(model "${KIPRJMOD}/Libraries/SynthStuff/3D_models/ALPHA-RD901F-40.step"
+			(offset
+				(xyz 7.35 -2.5 0)
+			)
+			(scale
+				(xyz 1 1 1)
+			)
+			(rotate
+				(xyz 0 0 90)
+			)
+		)
+		(model "${KIPRJMOD}/Libraries/SynthStuff/3D_models/rk09l12d0a1w.stp"
+			(hide yes)
+			(offset
+				(xyz 7.5 -2.5 6.7)
+			)
+			(scale
+				(xyz 1 1 1)
+			)
+			(rotate
+				(xyz 0 180 90)
+			)
+		)
