File: DMH_Mixer_PCB/DMH_Mixer_PCB.kicad_pcb (KiCad board)
At the start: 2 copper layers, 48 x 138 mm, 32 parts, among them J0 Conn_01x01, J100 IDC_02x05, J200 IDC_02x05, J50 Conn_01x08, J60 Conn_01x08, U1 TL074

Commit message: PCB redesign in progress
Parts:
- added RV5: 20k, Potentiometer_THT:Potentiometer_Bourns_3296W_Vertical, F.Cu at (93.8, 113.5)
- R8: value 1k -> 100k
- RV4: value 20k -> 100k
- moved J200 9.50 mm to (58.1, 153.2)
- moved RV4 8.14 mm to (72.5, 173.2)
Connections:
- J50 pad 5: /Core Circuit/Output - -> /Core Circuit/Output
- J50 pad 6: /Core Circuit/Output + -> /Core Circuit/Input 4
- R10 pad 2: Net-(R10-Pad2) -> Net-(U1D-+)
- R12 pad 1: Net-(R10-Pad2) -> Net-(U1D--)
- R4 pad 2: Net-(U1D-+) -> Net-(R4-Pad2)
- R5 pad 1: Net-(U1D-+) -> Net-(R4-Pad2)
- R7 pad 2: /Core Circuit/Output + -> /Core Circuit/Output
- R8 pad 1: Net-(U1D--) -> Net-(R8-Pad1)
- R8 pad 2: /Core Circuit/Output - -> Net-(U1A--)
- RV4 pad 2: GND -> Net-(R8-Pad1)
- RV4 pad 3: Net-(D1-K) -> /Core Circuit/Input 4
- U1 pad 1: Net-(U1D-+) -> Net-(R4-Pad2)
- U1 pad 8: Net-(R10-Pad2) -> Net-(U1D-+)
Routing:
- net (no net): track 0.00 -> 71.0 mm
- net Net-(R10-Pad2): track 62.0 -> 0.00 mm
- net Net-(D1-K): track 20.8 -> 5.50 mm
- net /Core Circuit/Input 3: track 49.5 -> 34.6 mm
- net /Core Circuit/Input 2: track 80.9 -> 66.9 mm
- net /Core Circuit/Output +: track 9.03 -> 0.00 mm
- net /Core Circuit/Output -: track 8.32 -> 0.00 mm
- net Net-(U1A--): track 41.1 -> 49.4 mm
- net Net-(J200-Pin_8): track 13.8 -> 5.53 mm
- net Net-(J200-Pin_7): track 13.8 -> 5.53 mm
- net Net-(J200-Pin_6): track 13.8 -> 5.53 mm
- net Net-(J200-Pin_1): track 16.3 -> 11.0 mm
- net Net-(J200-Pin_2): track 16.3 -> 14.7 mm
- net Net-(J200-Pin_3): track 16.3 -> 14.7 mm

Commit message: Rerouted main PCB
Parts:
- moved R8 40.2 mm to (65.0, 136.3), turned to 90 degrees
- moved R10 3.50 mm to (55.0, 136.3)
- moved R11 3.50 mm to (60.0, 128.7)
- moved R7 1.75 mm to (95.5, 164.2)
- moved C3 0.25 mm to (63.5, 103.2)
- moved C6 0.25 mm to (63.5, 124.8)
Routing:
- net (no net): track 71.0 -> 0.00 mm
- net Net-(D1-K): track 5.50 -> 67.0 mm
- net Net-(R8-Pad1): track 0.00 -> 41.1 mm
- net Net-(R4-Pad2): track 0.00 -> 33.0 mm
- net Net-(U1D-+): track 42.7 -> 19.0 mm
- net Net-(J200-Pin_8): track 5.53 -> 23.3 mm
- net Net-(J200-Pin_7): track 5.53 -> 23.3 mm
- net Net-(J200-Pin_6): track 5.53 -> 23.3 mm
- net Net-(U1A--): track 49.4 -> 65.3 mm
- net /Core Circuit/Input 4: track 0.00 -> 14.8 mm
- net Net-(J200-Pin_1): track 11.0 -> 25.8 mm
- net /Core Circuit/Input 3: track 34.6 -> 48.2 mm
- net /Core Circuit/Input 2: track 66.9 -> 80.1 mm
- net Net-(J200-Pin_2): track 14.7 -> 25.8 mm
- net Net-(J200-Pin_3): track 14.7 -> 25.8 mm
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
Commit message: Component placement ongoing
Parts:
- added R13: 33k, Resistor_THT:R_Axial_DIN0207_L6.3mm_D2.5mm_P7.62mm_Horizontal, F.Cu at (137.0, 114.0)
- added R14: 33k, Resistor_THT:R_Axial_DIN0207_L6.3mm_D2.5mm_P7.62mm_Horizontal, F.Cu at (137.0, 118.1)
- added R15: 33k, Resistor_THT:R_Axial_DIN0207_L6.3mm_D2.5mm_P7.62mm_Horizontal, F.Cu at (137.0, 122.1)
- added R16: 33k, Resistor_THT:R_Axial_DIN0207_L6.3mm_D2.5mm_P7.62mm_Horizontal, F.Cu at (137.0, 126.2)
- added SW1: SW_SPDT_321, SynthStuff:Toggle_Switch_THT, F.Cu at (128.9, 88.5)
- added SW2: SW_SPDT_321, SynthStuff:Toggle_Switch_THT, F.Cu at (137.6, 88.5)
- added SW3: SW_SPDT_321, SynthStuff:Toggle_Switch_THT, F.Cu at (146.2, 88.5)
- added SW4: SW_SPDT_321, SynthStuff:Toggle_Switch_THT, F.Cu at (154.9, 88.5)
- C1, C2, C3, C4, C5, C6, D1, D2, D4, D5, J100, J200, R1, R10, R11, R12, R2, R3, R4, R5, R6, R7, R8, R9, U1: moved to F.Cu
- moved C1 135.9 mm to (183.7, 92.9), turned to 0 degrees
- moved J0 133.3 mm to (183.7, 105.1)
- moved C4 123.7 mm to (174.8, 94.8), turned to 0 degrees
- moved D5 118.5 mm to (175.1, 87.5), turned to 0 degrees
- moved J200 114.8 mm to (166.5, 115.5), turned to 0 degrees
- moved C6 113.6 mm to (174.8, 101.7), turned to 0 degrees
- moved C3 111.9 mm to (174.8, 91.4), turned to 0 degrees
- moved C2 104.1 mm to (183.7, 99.5), turned to 0 degrees
- moved D4 94.7 mm to (175.1, 83.3), turned to 0 degrees
- moved J100 94.6 mm to (166.5, 87.3), turned to 0 degrees
- moved C5 88.9 mm to (174.8, 98.3), turned to 0 degrees
- moved R10 88.9 mm to (137.0, 101.9), turned to 0 degrees
- moved U1 83.9 mm to (148.2, 97.9), turned to 0 degrees
- moved R11 80.3 mm to (137.0, 105.9), turned to 0 degrees
- moved D2 72.8 mm to (147.7, 127.1)
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Connections:
- R10 pad 2: Net-(U1D-+) -> Net-(R10-Pad2)
- R12 pad 1: Net-(U1D--) -> Net-(R10-Pad2)
- R6 pad 2: Net-(R6-Pad2) -> Net-(U1D-+)
- R7 pad 1: Net-(R6-Pad2) -> Net-(U1D--)
- R9 pad 1: Net-(R6-Pad2) -> Net-(U1D-+)
- U1 pad 7: Net-(R6-Pad2) -> Net-(U1D-+)
- U1 pad 8: Net-(U1D-+) -> Net-(R10-Pad2)
Routing:
- net /Core Circuit/Input 1: track 127.0 -> 0.00 mm
- net -12V: track 122.8 -> 0.00 mm
- net Net-(R6-Pad2): track 83.3 -> 0.00 mm
- net /Core Circuit/Input 2: track 80.1 -> 0.00 mm
- net +12V: track 76.8 -> 0.00 mm
- net Net-(U1D--): track 76.2 -> 0.00 mm
- net Net-(D1-K): track 67.0 -> 0.00 mm
- net Net-(U1A--): track 65.3 -> 0.00 mm
- net Net-(SW3-C): track 58.6 -> 0.00 mm
- net Net-(D1-A): track 55.5 -> 0.00 mm
- net /Core Circuit/Input 3: track 48.2 -> 0.00 mm
- net Net-(SW4-C): track 41.1 -> 0.00 mm
- net Net-(R4-Pad2): track 33.0 -> 0.00 mm
- net Net-(SW2-C): track 27.8 -> 0.00 mm
- net Net-(J200-Pin_3): track 25.8 -> 0.00 mm
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- removed copper zone on B.Cu, net GND
- removed copper zone on F.Cu, net GND
