File: DMH_Mixer_PCB/DMH_Mixer_PCB.kicad_pcb (KiCad board)
At the start: 2 copper layers, 48 x 156 mm, 44 parts, among them J0 Conn_01x01, J100 IDC_02x05, J200 IDC_02x05, J50 Conn_01x08, J60 Conn_01x08, SW1 SW_SPDT_321, SW2 SW_SPDT_321, SW3 SW_SPDT_321, SW4 SW_SPDT_321, SW5 SW_DPDT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

Commit message: Prepared Gerbers for production
Other:
- board text added: "Mk1.0 - December 2024"
- board text removed: "Mk1.0 - Month Year"
Changed lines of the file:
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@@
 			(plot_on_all_layers_selection 0x0000000_00000000)
 			(disableapertmacros no)
-			(usegerberextensions no)
+			(usegerberextensions yes)
 			(usegerberattributes yes)
 			(usegerberadvancedattributes yes)
@@
 			(plotinvisibletext no)
 			(sketchpadsonfab no)
-			(subtractmaskfromsilk no)
+			(subtractmaskfromsilk yes)
 			(outputformat 1)
 			(mirror no)
-			(drillshape 1)
+			(drillshape 0)
 			(scaleselection 1)
-			(outputdirectory "")
+			(outputdirectory "Gerbers/")
 		)
 	)
@@
 		)
 		(fp_text user "${REFERENCE}"
-			(at 1.25 0 360)
+			(at 1.25 0 0)
 			(layer "B.Fab")
 			(effects
@@
 		(tags "Through hole vertical IDC box header THT 2x05 2.54mm double row")
 		(property "Reference" "J100"
-			(at -4.2475 3.67 -90)
+			(at -1.5 6.17 180)
 			(layer "B.SilkS")
 			(effects
@@
 		(attr through_hole)
 		(fp_line
-			(start -3.29 -15.37)
-			(end 5.83 -15.37)
+			(start -4.5 2.4)
+			(end -4.5 3.4)
 			(stroke
 				(width 0.12)
@@
 		)
 		(fp_line
-			(start -3.29 -7.13)
-			(end -1.98 -7.13)
+			(start -4.5 3.4)
+			(end -3.5 2.9)
 			(stroke
 				(width 0.12)
@@
 		)
 		(fp_line
-			(start -3.29 5.21)
-			(end -3.29 -15.37)
+			(start -3.5 2.9)
+			(end -4.5 2.4)
 			(stroke
 				(width 0.12)
@@
 		)
 		(fp_line
-			(start -3 -0.5)
-			(end -3 0.5)
+			(start -3.29 -15.37)
+			(end 5.83 -15.37)
 			(stroke
 				(width 0.12)
@@
 		)
 		(fp_line
-			(start -3 0.5)
-			(end -2 0)
+			(start -3.29 -7.13)
+			(end -1.98 -7.13)
 			(stroke
 				(width 0.12)
@@
 		)
 		(fp_line
-			(start -2 0)
-			(end -3 -0.5)
+			(start -3.29 5.21)
+			(end -3.29 -15.37)
 			(stroke
 				(width 0.12)
@@
 		)
 		(fp_text user "K"
-			(at 0 2.1 90)
+			(at 0.83 2 90)
 			(layer "B.SilkS")
 			(effects
@@
 		(tags "Resistor Axial_DIN0207 series Axial Horizontal pin pitch 7.62mm 0.25W = 1/4W length 6.3mm diameter 2.5mm")
 		(property "Reference" "R8"
-			(at 9.31 0 360)
+			(at 9.31 0 0)
 			(layer "B.SilkS")
 			(effects
@@
 		)
 		(property "Value" "100k"
-			(at 3.81 0 360)
+			(at 3.81 0 0)
 			(layer "B.SilkS")
 			(effects
@@
 		)
 		(fp_text user "${REFERENCE}"
-			(at 3.81 0 360)
+			(at 3.81 0 0)
 			(layer "B.Fab")
 			(effects
@@
 		)
 		(property "Value" "100k"
-			(at 3.81 0 360)
+			(at 3.81 0 0)
 			(layer "B.SilkS")
 			(effects
@@
 		)
 		(fp_text user "${REFERENCE}"
-			(at 3.81 0 360)
+			(at 3.81 0 0)
 			(layer "B.Fab")
 			(effects
@@
 		(tags "Resistor Axial_DIN0207 series Axial Horizontal pin pitch 7.62mm 0.25W = 1/4W length 6.3mm diameter 2.5mm")
 		(property "Reference" "R13"
-			(at -1.69 0 360)
+			(at -1.69 0 0)
 			(layer "B.SilkS")
 			(effects
@@
 		(tags "Resistor Axial_DIN0207 series Axial Horizontal pin pitch 7.62mm 0.25W = 1/4W length 6.3mm diameter 2.5mm")
 		(property "Reference" "R4"
-			(at 9.31 0 360)
+			(at 9.31 0 0)
 			(layer "B.SilkS")
 			(effects
@@
 		(tags "Resistor Axial_DIN0207 series Axial Horizontal pin pitch 7.62mm 0.25W = 1/4W length 6.3mm diameter 2.5mm")
 		(property "Reference" "R1"
-			(at 9.31 0 360)
+			(at 9.31 0 0)
 			(layer "B.SilkS")
 			(effects
@@
 		)
 		(property "Value" "1uF"
-			(at 2.5 0 360)
+			(at 2.5 0 0)
 			(layer "B.SilkS")
 			(effects
@@
 		)
 		(fp_text user "${REFERENCE}"
-			(at 2.5 0 360)
+			(at 2.5 0 0)
 			(layer "B.Fab")
 			(effects
@@
 		)
 		(property "Value" "1uF"
-			(at 2.5 0 360)
+			(at 2.5 0 0)
 			(layer "B.SilkS")
 			(effects
@@
 		)
 		(fp_text user "${REFERENCE}"
-			(at 2.5 0 360)
+			(at 2.5 0 0)
 			(layer "B.Fab")
 			(effects
@@
 		(tags "Resistor Axial_DIN0207 series Axial Horizontal pin pitch 7.62mm 0.25W = 1/4W length 6.3mm diameter 2.5mm")
 		(property "Reference" "R5"
-			(at 9.31 0 360)
+			(at 9.31 0 0)
 			(layer "B.SilkS")
 			(effects
@@
 		(tags "Resistor Axial_DIN0207 series Axial Horizontal pin pitch 7.62mm 0.25W = 1/4W length 6.3mm diameter 2.5mm")
 		(property "Reference" "R2"
-			(at 9.31 0 360)
+			(at 9.31 0 0)
 			(layer "B.SilkS")
 			(effects
@@
 		(tags "Diode DO-35_SOD27 series Axial Horizontal pin pitch 7.62mm  length 4mm diameter 2mm")
 		(property "Reference" "D3"
-			(at 9.41 0 360)
+			(at 9.41 0 0)
 			(layer "B.SilkS")
 			(effects
@@
 		(tags "Resistor Axial_DIN0207 series Axial Horizontal pin pitch 7.62mm 0.25W = 1/4W length 6.3mm diameter 2.5mm")
 		(property "Reference" "R10"
-			(at -1.69 0 360)
+			(at -1.69 0 0)
 			(layer "B.SilkS")
 			(effects
@@
 		(tags "Resistor Axial_DIN0207 series Axial Horizontal pin pitch 7.62mm 0.25W = 1/4W length 6.3mm diameter 2.5mm")
 		(property "Reference" "R3"
-			(at 9.31 0 360)
+			(at 9.31 0 0)
 			(layer "B.SilkS")
 			(effects
@@
 		)
 		(property "Value" "100nF"
-			(at 3 0 360)
+			(at 2 0 0)
 			(layer "B.SilkS")
 			(effects
@@
 		(tags "C Disc series Radial pin pitch 5.00mm  diameter 4.3mm width 1.9mm Capacitor")
 		(property "Reference" "C6"
-			(at -1.75 0 360)
+			(at -1.75 0 0)
 			(layer "B.SilkS")
 			(effects
@@
 		)
 		(property "Value" "100nF"
-			(at 3 0 90)
+			(at 2 0 90)
 			(layer "B.SilkS")
 			(effects
@@
 		(tags "Resistor Axial_DIN0207 series Axial Horizontal pin pitch 7.62mm 0.25W = 1/4W length 6.3mm diameter 2.5mm")
 		(property "Reference" "R6"
-			(at 9.31 0 360)
+			(at 9.31 0 0)
 			(layer "B.SilkS")
 			(effects
@@
 		)
 		(property "Value" "1uF"
-			(at 2.5 0 360)
+			(at 2.5 0 0)
 			(layer "B.SilkS")
 			(effects
@@
 		)
 		(fp_text user "${REFERENCE}"
-			(at 2.5 0 360)
+			(at 2.5 0 0)
 			(layer "B.Fab")
 			(effects
@@
 		)
 		(property "Value" "1uF"
-			(at 2.5 0 360)
+			(at 2.5 0 0)
 			(layer "B.SilkS")
 			(effects
@@
 		)
 		(fp_text user "${REFERENCE}"
-			(at 2.5 0 360)
+			(at 2.5 0 0)
 			(layer "B.Fab")
 			(effects
@@
 		(layer "User.9")
 	)
-	(gr_text "Mk1.0 - Month Year"
+	(gr_text "Mk1.0 - December 2024"
 		(at 97.5 131.5 90)
 		(layer "B.SilkS")
