File: DMH_Mixer_PCB/Inputs_and_Outputs.kicad_sch (KiCad schematic)
At the start: 0 parts

Commit message: PCB work in progress
Parts:
- added J1, J2, J3, J4, J5, J6: TS_Jack_6.35mm_Sw, SynthStuff:CUI_MJ-63052A, symbol SynthStuff:TS_Jack_6.35mm_Sw
- added J50, J51, J60, J61: Conn_01x06, Connector_PinHeader_2.54mm:PinHeader_1x06_P2.54mm_Vertical, symbol Connector_Generic:Conn_01x06
- added J7: IDC_02x05, SynthStuff:IDC-Header_2x05_P2.54mm_Vertical_BackBone, symbol SynthStuff:BackBone_Connector_10Pin
Connections:
- new net: J60.1 (Pin_1), J7.1 (Pin_1)
- new net: J60.2 (Pin_2), J7.2 (Pin_2)
- new net: J60.3 (Pin_3), J7.3 (Pin_3)
- new net: J60.4 (Pin_4), J7.6 (Pin_6)
- new net: J60.5 (Pin_5), J7.7 (Pin_7)
- new net: J60.6 (Pin_6), J7.8 (Pin_8)
- new net: J1.T, J51.1 (Pin_1)
- new net: J2.T, J51.2 (Pin_2)
- new net: J3.T, J51.3 (Pin_3)
- new net: J4.T, J51.4 (Pin_4)
- new net: J5.T, J51.5 (Pin_5)
- new net: J51.6 (Pin_6), J6.T
- new net: J1.TN, J61.1 (Pin_1)
- new net: J5.TN, J61.5 (Pin_5)
- new net: J2.TN, J61.2 (Pin_2)
- new net: J3.TN, J61.3 (Pin_3)
- new net: J4.TN, J61.4 (Pin_4)
- new net: J6.TN, J61.6 (Pin_6)
- new net GND: J1.S, J2.S, J3.S, J4.S, J5.S, J6.S, J7.10 (Pin_10), J7.4 (Pin_4), J7.5 (Pin_5), J7.9 (Pin_9)
- new net Input 1 Jack: J50.1 (Pin_1)
- new net Input 2 Jack: J50.2 (Pin_2)
- new net Input 3 Jack: J50.3 (Pin_3)
- new net Output + Jack: J50.5 (Pin_5)
- new net Output - Jack: J50.4 (Pin_4)
- new net Output Clipped: J50.6 (Pin_6)
Other:
- note added: "Not in main PCB"

Commit message: Component placing in progress
Parts:
- J51, J61: footprint Connector_PinHeader_2.54mm:PinHeader_1x06_P2.54mm_Vertical -> Connector_PinSocket_2.54mm:PinSocket_1x06_P2.54mm_Vertical
- renumbered J7 to J200
Changed lines of the file:
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@@
-	(wire
-		(pts
-			(xy 99.1149 53.34) (xy 99.1149 71.12)
-		)
-		(stroke
-			(width 0)
-			(type default)
-		)
-	)
 	(wire
 		(pts
@@
 	(wire
 		(pts
-			(xy 99.1149 71.12) (xy 121.92 71.12)
+			(xy 99.06 71.12) (xy 121.92 71.12)
 		)
 		(stroke
@@
 	(wire
 		(pts
-			(xy 43.18 53.34) (xy 99.1149 53.34)
-		)
-		(stroke
-			(width 0)
-			(type default)
-		)
-	)
-	(wire
-		(pts
 			(xy 50.8 99.06) (xy 50.8 73.66)
 		)
@@
 	(wire
 		(pts
+			(xy 99.06 53.34) (xy 99.06 71.12)
+		)
+		(stroke
+			(width 0)
+			(type default)
+		)
+	)
+	(wire
+		(pts
 			(xy 199.39 82.55) (xy 190.5 82.55)
 		)
@@
 		(pts
 			(xy 104.14 78.74) (xy 121.92 78.74)
+		)
+		(stroke
+			(width 0)
+			(type default)
+		)
+	)
+	(wire
+		(pts
+			(xy 43.18 53.34) (xy 99.06 53.34)
 		)
 		(stroke
@@
 			)
 		)
-		(property "Footprint" "Connector_PinHeader_2.54mm:PinHeader_1x06_P2.54mm_Vertical"
+		(property "Footprint" "Connector_PinSocket_2.54mm:PinSocket_1x06_P2.54mm_Vertical"
 			(at 127 121.92 0)
 			(effects
@@
 		(dnp no)
 		(fields_autoplaced yes)
-		(property "Reference" "J7"
+		(property "Reference" "J200"
 			(at 190.5 62.23 0)
 			(effects
@@
 				)
 				(hide yes)
+			)
+		)
+		(property "Function" ""
+			(at 190.5 73.66 0)
+			(effects
+				(font
+					(size 1.27 1.27)
+				)
 			)
 		)
@@
 			(project ""
 				(path "/58f4306d-5387-4983-bb08-41a2313fd315/ce3fef8b-9f1d-4178-b50b-4a046c030679"
-					(reference "J7")
+					(reference "J200")
 					(unit 1)
 				)
@@
 			)
 		)
-		(property "Footprint" "Connector_PinHeader_2.54mm:PinHeader_1x06_P2.54mm_Vertical"
+		(property "Footprint" "Connector_PinSocket_2.54mm:PinSocket_1x06_P2.54mm_Vertical"
 			(at 127 73.66 0)
 			(effects

Commit message: Finished main PCB
Parts:
- removed J51, J61: Conn_01x06, Connector_PinSocket_2.54mm:PinSocket_1x06_P2.54mm_Vertical, symbol Connector_Generic:Conn_01x06
- J50, J60: value Conn_01x06 -> Conn_01x08; footprint Connector_PinHeader_2.54mm:PinHeader_1x06_P2.54mm_Vertical -> Connector_PinSocket_2.54mm:PinSocket_1x08_P2.54mm_Vertical; symbol Connector_Generic:Conn_01x06 -> Connector_Generic:Conn_01x08
Connections:
- net GND: now also J50.7 (Pin_7), J50.8 (Pin_8), J60.7 (Pin_7), J60.8 (Pin_8)
- net Input 1 Jack: now also J1.T
- net Input 2 Jack: now also J2.T
- net Input 3 Jack: now also J3.T
- net Output + Jack: now also J5.T
- net Output - Jack: now also J4.T
- net Output Clipped: now also J6.T
- net at J200.1 (Pin_1), J60.1 (Pin_1): now also J1.TN
- net at J200.2 (Pin_2), J60.2 (Pin_2): now also J2.TN
- net at J200.3 (Pin_3), J60.3 (Pin_3): now also J3.TN
- net at J200.6 (Pin_6), J60.4 (Pin_4): now also J4.TN
- net at J200.7 (Pin_7), J60.5 (Pin_5): now also J5.TN
- net at J200.8 (Pin_8), J60.6 (Pin_6): now also J6.TN

Commit message: Added 4th channel to schematic
... and replaced Inverted Output with Clipped Output
Parts:
- J1: Function Input 1 -> In 1
- J2: Function Input 2 -> In 2
- J3: Function Input 3 -> In 3
- J4: Function Output - -> Clip
- J5: Function Output + -> Out
- J6: Function Clipped Output -> In 4
Connections:
- net Output + Jack renamed Output Jack
- net Output - Jack renamed Clipped Output Jack
- net Output Clipped renamed Input 4 Jack
Other:
- note added: "Connectors PCB"
- note removed: "Not in main PCB"
Changed lines of the file:
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@@
 		)
 	)
-	(text "Not in main PCB"
+	(text "Connectors PCB"
 		(exclude_from_sim no)
 		(at 130.556 172.212 0)
@@
 		)
 	)
-	(hierarchical_label "Output Clipped"
-		(shape input)
+	(hierarchical_label "Input 4 Jack"
+		(shape output)
 		(at 165.1 129.54 0)
 		(fields_autoplaced yes)
@@
 		)
 	)
-	(hierarchical_label "Output - Jack"
+	(hierarchical_label "Clipped Output Jack"
 		(shape input)
 		(at 165.1 124.46 0)
@@
 		)
 	)
-	(hierarchical_label "Output + Jack"
+	(hierarchical_label "Output Jack"
 		(shape input)
 		(at 165.1 127 0)
@@
 			)
 		)
-		(property "Function" "Input 1"
+		(property "Function" "In 1"
 			(at 38.1 33.02 0)
 			(effects
@@
 			)
 		)
-		(property "Function" "Output +"
+		(property "Function" "Out"
 			(at 38.1 134.874 0)
 			(effects
@@
 			)
 		)
-		(property "Function" "Input 2"
+		(property "Function" "In 2"
 			(at 38.1 58.42 0)
 			(effects
@@
 			)
 		)
-		(property "Function" "Input 3"
+		(property "Function" "In 3"
 			(at 38.1 83.82 0)
 			(effects
@@
 			)
 		)
-		(property "Function" "Output -"
+		(property "Function" "Clip"
 			(at 38.1 109.474 0)
 			(effects
@@
 			)
 		)
-		(property "Function" "Clipped Output"
+		(property "Function" "In 4"
 			(at 38.354 160.274 0)
 			(effects

Commit message: Moved output jacks to bottom right
Parts:
- renumbered J6 to J4, J4 to J5, J5 to J6
Connections:
- net Clipped Output Jack: now also J50.5 (Pin_5); no longer J50.4 (Pin_4)
- net Input 4 Jack: now also J50.4 (Pin_4); no longer J50.6 (Pin_6)
- net Output Jack: now also J50.6 (Pin_6); no longer J50.5 (Pin_5)
- net at J200.6 (Pin_6), J60.4 (Pin_4): now also J4.TN; no longer J5.TN
- net at J200.7 (Pin_7), J60.5 (Pin_5): now also J5.TN; no longer J6.TN
- net at J200.8 (Pin_8), J60.6 (Pin_6): now also J6.TN; no longer J4.TN
Other:
- moved on the sheet: J4, J5, J6

Commit message: Finalization in progress
Parts:
- removed J6: TS_Jack_6.35mm_Sw, SynthStuff:CUI_MJ-63052A, symbol SynthStuff:TS_Jack_6.35mm_Sw
- J5: Function Clip -> Out
Connections:
- net Clipped Output Jack is gone; now on net Output Jack: J5.T, J50.5 (Pin_5)
- net Output Jack: no longer J50.6 (Pin_6)
- net at J60.6 (Pin_6): no longer J200.8 (Pin_8)
Changed lines of the file:
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@@
-	)
-	(junction
-		(at 157.48 81.28)
-		(diameter 0)
-		(color 0 0 0 0)
 	)
 	(junction
@@
 	)
 	(junction
-		(at 157.48 129.54)
-		(diameter 0)
-		(color 0 0 0 0)
-	)
-	(junction
 		(at 157.48 124.46)
 		(diameter 0)
@@
 	)
 	(junction
-		(at 50.8 149.86)
-		(diameter 0)
-		(color 0 0 0 0)
-	)
-	(junction
 		(at 132.08 134.62)
 		(diameter 0)
@@
 	(wire
 		(pts
-			(xy 50.8 149.86) (xy 50.8 165.1)
-		)
-		(stroke
-			(width 0)
-			(type default)
-		)
-	)
-	(wire
-		(pts
-			(xy 173.99 90.17) (xy 207.01 90.17)
-		)
-		(stroke
-			(width 0)
-			(type default)
-		)
-	)
-	(wire
-		(pts
 			(xy 43.18 127) (xy 157.48 127)
 		)
@@
 	(wire
 		(pts
-			(xy 43.18 149.86) (xy 50.8 149.86)
-		)
-		(stroke
-			(width 0)
-			(type default)
-		)
-	)
-	(wire
-		(pts
 			(xy 50.8 22.86) (xy 50.8 48.26)
 		)
@@
 	(wire
 		(pts
-			(xy 43.18 152.4) (xy 109.22 152.4)
-		)
-		(stroke
-			(width 0)
-			(type default)
-		)
-	)
-	(wire
-		(pts
-			(xy 207.01 73.66) (xy 196.85 73.66)
-		)
-		(stroke
-			(width 0)
-			(type default)
-		)
-	)
-	(wire
-		(pts
 			(xy 99.06 78.74) (xy 99.06 73.66)
 		)
@@
 	(wire
 		(pts
-			(xy 157.48 129.54) (xy 165.1 129.54)
-		)
-		(stroke
-			(width 0)
-			(type default)
-		)
-	)
-	(wire
-		(pts
 			(xy 43.18 73.66) (xy 50.8 73.66)
 		)
@@
 	(wire
 		(pts
-			(xy 207.01 90.17) (xy 207.01 73.66)
-		)
-		(stroke
-			(width 0)
-			(type default)
-		)
-	)
-	(wire
-		(pts
 			(xy 176.53 87.63) (xy 204.47 87.63)
 		)
@@
 	(wire
 		(pts
-			(xy 50.8 124.46) (xy 50.8 149.86)
+			(xy 50.8 124.46) (xy 50.8 165.1)
 		)
 		(stroke
@@
 	(wire
 		(pts
-			(xy 106.68 81.28) (xy 157.48 81.28)
-		)
-		(stroke
-			(width 0)
-			(type default)
-		)
-	)
-	(wire
-		(pts
 			(xy 50.8 99.06) (xy 50.8 124.46)
 		)
@@
 	(wire
 		(pts
-			(xy 157.48 81.28) (xy 173.99 81.28)
-		)
-		(stroke
-			(width 0)
-			(type default)
-		)
-	)
-	(wire
-		(pts
 			(xy 199.39 78.74) (xy 199.39 82.55)
 		)
@@
 	(wire
 		(pts
-			(xy 109.22 129.54) (xy 157.48 129.54)
-		)
-		(stroke
-			(width 0)
-			(type default)
-		)
-	)
-	(wire
-		(pts
 			(xy 184.15 78.74) (xy 181.61 78.74)
 		)
@@
 	(wire
 		(pts
-			(xy 109.22 152.4) (xy 109.22 129.54)
-		)
-		(stroke
-			(width 0)
-			(type default)
-		)
-	)
-	(wire
-		(pts
 			(xy 76.2 116.84) (xy 157.48 116.84)
 		)
@@
 	(wire
 		(pts
-			(xy 43.18 154.94) (xy 106.68 154.94)
-		)
-		(stroke
-			(width 0)
-			(type default)
-		)
-	)
-	(wire
-		(pts
 			(xy 157.48 121.92) (xy 165.1 121.92)
 		)
@@
 	(wire
 		(pts
-			(xy 173.99 81.28) (xy 173.99 90.17)
-		)
-		(stroke
-			(width 0)
-			(type default)
-		)
-	)
-	(wire
-		(pts
 			(xy 101.6 76.2) (xy 157.48 76.2)
-		)
-		(stroke
-			(width 0)
-			(type default)
-		)
-	)
-	(wire
-		(pts
-			(xy 106.68 154.94) (xy 106.68 81.28)
 		)
 		(stroke
@@
 		)
 	)
-	(hierarchical_label "Clipped Output Jack"
+	(hierarchical_label "Output Jack"
 		(shape input)
 		(at 165.1 127 0)
@@
 		(shape output)
 		(at 165.1 119.38 0)
-		(fields_autoplaced yes)
-		(effects
-			(font
-				(size 1.27 1.27)
-			)
-			(justify left)
-		)
-	)
-	(hierarchical_label "Output Jack"
-		(shape input)
-		(at 165.1 129.54 0)
 		(fields_autoplaced yes)
 		(effects
@@
 	(symbol
 		(lib_id "SynthStuff:TS_Jack_6.35mm_Sw")
-		(at 38.1 152.4 0)
-		(unit 1)
-		(exclude_from_sim no)
-		(in_bom yes)
-		(on_board no)
-		(dnp no)
-		(property "Reference" "J6"
-			(at 37.465 143.51 0)
-			(effects
-				(font
-					(size 1.27 1.27)
-				)
-			)
-		)
-		(property "Value" "TS_Jack_6.35mm_Sw"
-			(at 37.465 146.05 0)
-			(effects
-				(font
-					(size 1.27 1.27)
-				)
-			)
-		)
-		(property "Footprint" "SynthStuff:CUI_MJ-63052A"
-			(at 38.1 152.4 0)
-			(effects
-				(font
-					(size 1.27 1.27)
-				)
-				(hide yes)
-			)
-		)
-		(property "Datasheet" "~"
-			(at 38.1 152.4 0)
-			(effects
-				(font
-					(size 1.27 1.27)
-				)
-				(hide yes)
-			)
-		)
-		(property "Description" "Audio Jack, 2 Poles (Mono / TS), Switched T Pole (Normalling), 6.35mm, 1/4inch"
-			(at 38.1 152.4 0)
-			(effects
-				(font
-					(size 1.27 1.27)
-				)
-				(hide yes)
-			)
-		)
-		(property "Function" "Out"
-			(at 38.1 160.274 0)
-			(effects
-				(font
-					(size 1.27 1.27)
-					(thickness 0.254)
-					(bold yes)
-					(italic yes)
-				)
-			)
-		)
-		(pin "T"
-		)
-		(pin "TN"
-		)
-		(pin "S"
-		)
-		(instances
-			(project ""
-				(path "/58f4306d-5387-4983-bb08-41a2313fd315/ce3fef8b-9f1d-4178-b50b-4a046c030679"
-					(reference "J6")
-					(unit 1)
-				)
-			)
-		)
-	)
-	(symbol
-		(lib_id "SynthStuff:TS_Jack_6.35mm_Sw")
 		(at 38.1 50.8 0)
 		(unit 1)
@@
 			)
 		)
-		(property "Function" "Clip"
+		(property "Function" "Out"
 			(at 38.1 134.874 0)
 			(effects

Commit message: Finalized schematic
Connections:
- no-connect marks 0 -> 3
Changed lines of the file:
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@@
 		(color 0 0 0 0)
+	)
+	(no_connect
+		(at 196.85 73.66)
+	)
+	(no_connect
+		(at 157.48 81.28)
+	)
+	(no_connect
+		(at 157.48 129.54)
 	)
 	(wire
