File: DMH_Mixer_PCB/Power.kicad_sch (KiCad schematic)
At the start: 14 parts, among them J0 Conn_01x01, J100 IDC_02x08, J101 IDC_02x05

Commit message: PCB work in progress
Parts:
- removed C3: 47uF, Capacitor_THT:CP_Radial_D4.0mm_P1.50mm, symbol Device:C_Polarized
- removed D1, D3: SB140+, Diode_THT:D_DO-41_SOD81_P10.16mm_Horizontal, symbol SynthStuff:Power_Bus_Schotty_+
- removed D2: SB140-, Diode_THT:D_DO-41_SOD81_P10.16mm_Horizontal, symbol SynthStuff:Power_Bus_Schotty_-
- removed J100: IDC_02x08, SynthStuff:IDC-Header_2x08_P2.54mm_Vertical_Eurorack, symbol SynthStuff:Eurorack_Power_Connector_16Pin
- added C3: 100nF, Capacitor_THT:C_Disc_D4.3mm_W1.9mm_P5.00mm, symbol Device:C
- added U1: TL074, Package_DIP:DIP-14_W7.62mm_Socket, symbol Amplifier_Operational:TL074
- renumbered J101 to J100
Connections:
- net +5V is gone; now on net GND: C6.1
- net +12V: now also C3.1, U1.4 (V+)
- net -12V: now also C6.2, U1.11 (V-)
- net GND: now also C3.2; no longer C6.2
Other:
- note removed: "Delete what's not needed!"

Commit message: Finalized schematic
Parts:
- removed U1: TL074, Package_DIP:DIP-14_W7.62mm_Socket, symbol Amplifier_Operational:TL074
- added U1: TL072, symbol Amplifier_Operational:TL072
- renumbered C4 to C3, C5 to C4, C3 to C5, D5 to D1, D4 to D2
Connections:
- net +12V: now also U1.8 (V+)
- net -12V: now also U1.4 (V-)
