File: DMH_Mixer_PANEL/DMH_Mixer_PANEL.kicad_pcb (KiCad board)
At the start: 2 copper layers, 50 x 200 mm, 15 parts, among them J0 Panel_GND_Solder_Wire_Pad

Commit message: Replaced clipping with 4th channel on panel
Parts:
- removed H10: Clip, SynthStuff:Jack_6.35mm_Cutout_Output_v6
- removed H14: Clip, SynthStuff:Pot_Cutout_Tiny
- added H15: Input 4, SynthStuff:Jack_6.35mm_Cutout_v3, F.Cu at (91.5, 208.8)
- added H16: Input 4 Gain, SynthStuff:Pot_Cutout_Small, F.Cu at (75.0, 165.8)
- H5: value In 1 -> Input 1
- H6: value In 2 -> Input 2
- H7: value In 3 -> Input 3

Commit message: Added 4th channel to schematic
... and replaced Inverted Output with Clipped Output
Parts:
- H15: value Input 4 -> In 4
- H5: value Input 1 -> In 1
- H6: value Input 2 -> In 2
- H7: value Input 3 -> In 3
- H8: value Out + -> Out
- H9: value Out - -> Clip

Commit message: PCB redesign in progress
Parts:
- added H10: Clip Amt, SynthStuff:MountingHole_TrimPot, F.Cu at (95.0, 112.5)
Changed lines of the file:
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@@
+		)
+	)
+	(footprint "SynthStuff:MountingHole_TrimPot"
+		(layer "F.Cu")
+		(at 95 112.5)
+		(descr "Mounting Hole 2.5mm, no annular")
+		(tags "mounting hole 2.5mm no annular")
+		(property "Reference" "H10"
+			(at 0 -3.5 0)
+			(layer "F.Fab")
+			(effects
+				(font
+					(size 1 1)
+					(thickness 0.15)
+				)
+			)
+		)
+		(property "Value" "Clip Amt"
+			(at 0 3.5 0)
+			(layer "F.SilkS")
+			(effects
+				(font
+					(size 1 1)
+					(thickness 0.15)
+				)
+			)
+		)
+		(property "Footprint" "SynthStuff:MountingHole_TrimPot"
+			(at 0 0 0)
+			(unlocked yes)
+			(layer "F.Fab")
+			(hide yes)
+			(effects
+				(font
+					(size 1.27 1.27)
+					(thickness 0.15)
+				)
+			)
+		)
+		(property "Datasheet" ""
+			(at 0 0 0)
+			(unlocked yes)
+			(layer "F.Fab")
+			(hide yes)
+			(effects
+				(font
+					(size 1.27 1.27)
+					(thickness 0.15)
+				)
+			)
+		)
+		(property "Description" "Mounting Hole Trimpot"
+			(at 0 0 0)
+			(unlocked yes)
+			(layer "F.Fab")
+			(hide yes)
+			(effects
+				(font
+					(size 1.27 1.27)
+					(thickness 0.15)
+				)
+			)
+		)
+		(property ki_fp_filters "MountingHole*")
+		(sheetname "Root")
+		(sheetfile "DMH_Mixer_PANEL.kicad_sch")
+		(attr exclude_from_pos_files exclude_from_bom)
+		(fp_circle
+			(center 0 0)
+			(end 2.5 0)
+			(stroke
+				(width 0.15)
+				(type solid)
+			)
+			(fill none)
+			(layer "Cmts.User")
+		)
+		(fp_circle
+			(center 0 0)
+			(end 2.75 0)
+			(stroke
+				(width 0.05)
+				(type solid)
+			)
+			(fill none)
+			(layer "F.CrtYd")
+		)
+		(fp_text user "${REFERENCE}"
+			(at 0 0 0)
+			(layer "F.Fab")
+			(effects
+				(font
+					(size 1 1)
+					(thickness 0.15)
+				)
+			)
+		)
+		(pad "" np_thru_hole circle
+			(at 0 0)
+			(size 2.5 2.5)
+			(drill 2.5)
+			(layers "*.Cu" "*.Mask")
+		)
+		(model "${KICAD8_3DMODEL_DIR}/Potentiometer_THT.3dshapes/Potentiometer_Bourns_3296W_Vertical.step"
+			(offset
+				(xyz -1.1 -1 -11.8)
+			)
+			(scale
+				(xyz 1 1 1)
+			)
+			(rotate
+				(xyz 0 0 -90)
+			)
 		)
 	)
@@
 		(layer "Dwgs.User")
 	)
+	(gr_line
+		(start 75 94.25)
+		(end 75 130)
+		(stroke
+			(width 0.1)
+			(type default)
+		)
+		(layer "Cmts.User")
+	)
+	(gr_line
+		(start 75 58.5)
+		(end 75 94.25)
+		(stroke
+			(width 0.1)
+			(type default)
+		)
+		(layer "Cmts.User")
+	)
+	(gr_circle
+		(center 75 76.375)
+		(end 95 76.4)
+		(stroke
+			(width 0.1)
+			(type default)
+		)
+		(fill none)
+		(layer "Cmts.User")
+	)
+	(gr_circle
+		(center 75 112.125)
+		(end 95 112.15)
+		(stroke
+			(width 0.1)
+			(type default)
+		)
+		(fill none)
+		(layer "Cmts.User")
+	)
 	(gr_rect

Commit message: Added toggle switches to front panel
Parts:
- added H14: Input 1 Line/10Vpp, SynthStuff:Toggle_Switch_Cutout, F.Cu at (58.5, 58.5)
- added H17: Input 2 Line/10Vpp, SynthStuff:Toggle_Switch_Cutout, F.Cu at (58.5, 94.2)
- added H18: Input 3 Line/10Vpp, SynthStuff:Toggle_Switch_Cutout, F.Cu at (58.5, 130.0)
- added H19: Input 4 Line/10Vpp, SynthStuff:Toggle_Switch_Cutout, F.Cu at (58.5, 165.8)
- moved H10 40.0 mm to (55.0, 112.5)
- moved J0 18.3 mm to (56.8, 148.2)
- moved H11 8.00 mm to (83.0, 58.5)
- moved H12 8.00 mm to (83.0, 94.2)
- moved H13 8.00 mm to (83.0, 130.0)
- moved H16 8.00 mm to (83.0, 165.8)
Other:
- board text added: "Euro"
- board text added: "Line"

Commit message: Component placement ongoing
Parts:
- moved J0 1.75 mm to (55.0, 148.2)
Changed lines of the file:
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@@
 	(footprint "SynthStuff:Panel_GND_SolderWirePad_5x10mm"
 		(layer "B.Cu")
-		(at 56.75 148.25 180)
+		(at 55 148.25 180)
 		(descr "Wire Pad, Square, SMD Pad,  5mm x 10mm,")
 		(tags "MesurementPoint Square SMDPad 5mmx10mm ")

Commit message: Moved pots to X=83,25
Parts:
- moved H11 0.25 mm to (83.2, 58.5)
- moved H12 0.25 mm to (83.2, 94.2)
- moved H13 0.25 mm to (83.2, 130.0)
- moved H16 0.25 mm to (83.2, 165.8)
Other:
- board text added: "Euro (DC)"
- board text added: "Line (AC)"
- board text removed: "Euro"
- board text removed: "Line"

Commit message: ReRouted PCB
Other:
- board text added: "Audio & CV"
- board text removed: "DC Coupled"

Commit message: Moved output jacks to bottom right
Parts:
- moved H15 33.0 mm to (58.5, 208.8)
- moved H8 16.5 mm to (91.5, 208.8)
- moved H9 16.5 mm to (75.0, 208.8)
